File: Board/PY32F071R1BU6_EB/untitled.kicad_sch (KiCad schematic)
At the start: 0 parts

Commit message: Display added to schematic
Parts:
- added C1: 1uF, Capacitor_SMD:C_0603_1608Metric_Pad1.08x0.95mm_HandSolder, symbol Device:C
- added J5: Conn_01x08, Connector_PinSocket_2.54mm:PinSocket_1x08_P2.54mm_Vertical, symbol Connector_Generic:Conn_01x08
- added Q1: IRLML0030, Package_TO_SOT_SMD:SOT-23, symbol Transistor_FET:IRLML0030
- added R13: 10k, Resistor_SMD:R_0603_1608Metric_Pad0.98x0.95mm_HandSolder, symbol Device:R
- added R14: 1k, Resistor_SMD:R_0603_1608Metric_Pad0.98x0.95mm_HandSolder, symbol Device:R
- added U5: ST7735S_13P, USER:ST7735S_13P_0.96IN_80X160, symbol USER:ST7735S_13P
Connections:
- new net: Q1.1 (G), R13.2, R14.2
- new net +3V3: C1.1, J5.2 (Pin_2), R13.1
- new net BLK: J5.8 (Pin_8), R14.1
- new net CSX: J5.7 (Pin_7)
- new net D0: J5.4 (Pin_4)
- new net DCX: J5.6 (Pin_6)
- new net GND: C1.2, J5.1 (Pin_1), Q1.2 (S)
- new net RESX: J5.5 (Pin_5)
- new net SCL: J5.3 (Pin_3)

Commit message: Schematic updated
Parts:
- added C7, C8, C9: 100nF, Capacitor_SMD:C_0603_1608Metric_Pad1.08x0.95mm_HandSolder, symbol Device:C
- added D1, D3, D4: LED, LED_SMD:LED_0603_1608Metric, symbol Device:LED
- added D5: BAT54S, Package_TO_SOT_SMD:SOT-23, symbol Diode:BAT54S
- added J6: Conn_Coaxial, Connector_Coaxial:U.FL_Hirose_U.FL-R-SMT-1_Vertical, symbol Connector:Conn_Coaxial
- added J7: Conn_01x03, Connector_PinHeader_2.54mm:PinHeader_1x03_P2.54mm_Vertical, symbol Connector_Generic:Conn_01x03
- added R15: 10R, Resistor_SMD:R_0603_1608Metric_Pad0.98x0.95mm_HandSolder, symbol Device:R
- added R16, R18, R19: 510R, Resistor_SMD:R_0603_1608Metric_Pad0.98x0.95mm_HandSolder, symbol Device:R
- added R17, R23, R24: 10k, Resistor_SMD:R_0603_1608Metric_Pad0.98x0.95mm_HandSolder, symbol Device:R
- added R20, R21, R22: 1k, Resistor_SMD:R_0603_1608Metric_Pad0.98x0.95mm_HandSolder, symbol Device:R
- added R25: 100R, Resistor_SMD:R_0603_1608Metric_Pad0.98x0.95mm_HandSolder, symbol Device:R
- added R26, R27: 1M, Resistor_SMD:R_0603_1608Metric_Pad0.98x0.95mm_HandSolder, symbol Device:R
- added SW1: BTN0, USER:SW_SPST_CK_PTS641, symbol Switch:SW_Push
- added SW2: BTN1, USER:SW_SPST_CK_PTS641, symbol Switch:SW_Push
- added SW3: BTN2, USER:SW_SPST_CK_PTS641, symbol Switch:SW_Push
Connections:
- net +3V3: now also U5.10 (Pin_10), U5.12 (Pin_12), D5.2 (K), R16.1, R17.1, R18.1, R19.1, R23.1, R24.1, R26.1
- net BTN0: now also C7.1, R20.1
- net BTN1: now also C9.1, R21.1
- net BTN2: now also C8.1, R22.1
- net CSX: now also U5.7 (Pin_7)
- net D0: now also U5.4 (Pin_4)
- net DCX: now also U5.5 (Pin_5)
- net GND: now also U5.13 (Pin_13), U5.8 (Pin_8), C7.2, C8.2, C9.2, D5.1 (A), J6.2 (Ext), J7.1 (Pin_1), J7.3 (Pin_3), R27.2, SW1.2, SW2.2, SW3.2
- net LED0: now also D1.1 (K)
- net LED1: now also D3.1 (K)
- net LED2: now also D4.1 (K)
- net RESX: now also U5.6 (Pin_6)
- net SCL: now also U5.3 (Pin_3)
- net at Q1.3 (D): now also R15.2
- net at U5.11 (Pin_11): now also R15.1
- new net: D4.2 (A), R19.2
- new net: D1.2 (A), R16.2
- new net: R22.2, R24.2, SW3.1
- new net: R21.2, R23.2, SW2.1
- new net: R17.2, R20.2, SW1.1
- new net: J6.1 (In), J7.2 (Pin_2), R25.2
- new net: D3.2 (A), R18.2
- new net FREQ: D5.3 (COM), R25.1, R26.2, R27.1
Other:
- note added: "CS"
- note added: "GND"
- note added: "LED+"
- note added: "LED-"
- note added: "NC"
- note added: "RESET"
- note added: "RS"
- note added: "SCL"
- note added: "SDA"
- note added: "TP0"
- note added: "TP1"
- note added: "VCC"
- moved on the sheet: C1, J5, Q1, R13, R14, U5

Commit message: Component placement started
Parts:
- D5: footprint Package_TO_SOT_SMD:SOT-23 -> Package_TO_SOT_SMD:SOT-23-3
Changed lines of the file:
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@@
 			)
 		)
-		(property "Footprint" "Package_TO_SOT_SMD:SOT-23"
+		(property "Footprint" "Package_TO_SOT_SMD:SOT-23-3"
 			(at 55.245 38.735 0)
 			(effects
